File: Drive/PCB/ESP32-S3.kicad_sch (KiCad schematic)
At the start: 17 parts, among them IC5 ESP32-S3-WROOM-1U-N8, J10 USB_C_Receptacle_USB2.0_16P, SW1 SW_Push, SW2 SW_Push, U1 USBLC6-2SC6, U2 AMS1117-3.3

Commit message: Adds V2.1 Driver Files
Parts:
- removed C13: 22u, Capacitor_SMD:C_1206_3216Metric, symbol Device:C
- removed IC5: ESP32-S3-WROOM-1U-N8, Footprints:ESP32S3WROOM1UN8, symbol ESP_SMD:ESP32-S3-WROOM-1U-N8
- added C13: TAJB226K020RNJ, CAPPM3528X210N, symbol Capacitor_2:TAJB226K020RNJ
- added C15: 100n, Capacitor_SMD:C_0402_1005Metric, symbol Device:C
- added IC5: ESP32-C6-MINI-1U-N4, ESP32C6MINI1UN4, symbol ESP_SMD:ESP32-C6-MINI-1U-N4
- added R26, R27: 22, Resistor_SMD:R_0402_1005Metric, symbol Device:R
- C14: value 100n -> 22u; footprint Capacitor_SMD:C_0402_1005Metric -> Capacitor_SMD:C_1206_3216Metric
Connections:
- net 3V3: now also C13.1 (+), C15.1, IC5.3 (3V3); no longer C12.1 (+)
- net 5V: now also C12.1 (+)
- net BOOT: now also IC5.23 (IO9)
- net D+: now also R27.2
- net D-: now also R26.2
- net GND: now also C13.2 (-), C15.2, IC5.1 (GND_1), IC5.11 (GND_3), IC5.14 (GND_4), IC5.2 (GND_2), IC5.36 (GND_5), IC5.37 (GND_6), IC5.38 (GND_7), IC5.39 (GND_8), IC5.40 (GND_9), IC5.41 (GND_10), IC5.42 (GND_11), IC5.43 (GND_12), IC5.44 (GND_13), IC5.45 (GND_14), IC5.46 (GND_15), IC5.47 (GND_16), IC5.48 (GND_17), IC5.49 (GND_18), IC5.50 (GND_19), IC5.51 (GND_20), IC5.52 (GND_21), IC5.53 (GND_22), IC5.54 (GND_23), IC5.55 (GND_24), IC5.56 (GND_25), IC5.57 (GND_26), IC5.58 (GND_27), IC5.59 (GND_28), IC5.60 (GND_29), IC5.61 (GND_30)
- net GPIO1: now also IC5.13 (IO1)
- net GPIO15: now also IC5.20 (IO15)
- net GPIO16: now also IC5.31 (TXD0)
- net GPIO17: now also IC5.30 (RXD0)
- net GPIO18: now also IC5.24 (IO18)
- net GPIO2: now also IC5.5 (IO2)
- net GPIO21: now also IC5.27 (IO21)
- net GPIO3: now also IC5.6 (IO3)
- net GPIO4: now also IC5.9 (IO4)
- net GPIO5: now also IC5.10 (IO5)
- net GPIO6: now also IC5.15 (IO6)
- net GPIO7: now also IC5.16 (IO7)
- net GPIO8: now also IC5.22 (IO8)
- net RST: now also IC5.8 (EN)
- net USB_D+: now also U1.3 (I/O2); no longer J10.A6 (D+), U1.1 (I/O1)
- net USB_D-: now also U1.1 (I/O1); no longer J10.A7 (D-), U1.3 (I/O2)
- new net DR+: IC5.18 (IO13), R27.1
- new net DR-: IC5.17 (IO12), R26.1
- new net GPIO0: IC5.12 (IO0)
- new net GPIO19: IC5.25 (IO19)
- new net GPIO20: IC5.26 (IO20)
- new net GPIO22: IC5.28 (IO22)
- new net GPIO23: IC5.29 (IO23)
- no-connect marks 2 -> 10
