File: Drive/PCB/Odyssey_Driver.kicad_sch (KiCad schematic)
At the start: 1 part, among them J1 Conn_01x02

Commit message: Adds V2.1 Driver Files
Connections:
- no-connect marks 17 -> 0
Other:
- sheet ESP32-S3 renamed ESP32-C6
- sheet ESP32-C6 ports: added 3V3, GPIO0, GPIO19, GPIO20, GPIO22, GPIO23; removed GPIO10, GPIO11, GPIO12, GPIO13, GPIO14, GPIO35, GPIO36, GPIO37, GPIO38, GPIO39, GPIO40, GPIO41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
