File: Drive/PCB/Odyssey_Driver.kicad_pcb (KiCad board)
At the start: 4 copper layers, 100 x 80 mm, 81 parts, among them IC1 L298N, IC2 PCA9546ADR, IC3 L298N, IC4 ADS1015BQDGSRQ1, IC5 ESP32-S3-WROOM-1U-N8, J1 Conn_01x02, J10 USB_C_Receptacle_USB2.0_16P, J2 Conn_01x02, J3 Conn_01x02, J4 Conn_01x04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

Commit message: Adds V2.1 Driver Files
Parts:
- added C15: 100n, Capacitor_SMD:C_0402_1005Metric, F.Cu at (161.0, 118.1)
- added R26: 22, Resistor_SMD:R_0402_1005Metric, F.Cu at (166.5, 110.9)
- added R27: 22, Resistor_SMD:R_0402_1005Metric, F.Cu at (166.5, 109.8)
- C1, C2, C6, C7: value EEHZT1E331UP -> HV1E477M0810PZ
- C13: value 22u -> TAJB226K020RNJ; footprint Capacitor_SMD:C_1206_3216Metric -> Footprints:CAPPM3528X210N
- C14: value 100n -> 22u; footprint Capacitor_SMD:C_0402_1005Metric -> Capacitor_SMD:C_1206_3216Metric
- IC5: value ESP32-S3-WROOM-1U-N8 -> ESP32-C6-MINI-1U-N4; footprint Footprints:ESP32S3WROOM1UN8 -> Footprints:ESP32C6MINI1UN4
- moved D19 55.8 mm to (124.8, 117.2), turned to 0 degrees
- moved D20 53.6 mm to (124.8, 118.4), turned to 0 degrees
- moved R21 52.8 mm to (127.5, 117.2), turned to 0 degrees
- moved R22 50.7 mm to (127.5, 118.4), turned to 0 degrees
- moved C11 36.7 mm to (132.9, 119.6)
- moved R20 33.5 mm to (134.1, 118.6)
- moved SW1 25.3 mm to (140.1, 118.7)
- moved C14 14.5 mm to (159.1, 119.4)
- moved C12 12.5 mm to (176.7, 114.3), turned to 180 degrees
- moved J10 10.9 mm to (186.8, 119.8), turned to 0 degrees
- moved C13 9.88 mm to (168.6, 118.4), turned to 90 degrees
- moved SW2 8.32 mm to (136.5, 118.7)
- moved U1 7.71 mm to (171.7, 110.3)
- moved R23 6.10 mm to (184.2, 114.1), turned to 180 degrees
- moved REF** 6.00 mm to (196.0, 120.0)
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Connections:
- net /ESP32-S3/GPIO37 renamed /ESP32-C6/GPIO17
- C11 pad 1: /ESP32-S3/RST -> /ESP32-C6/RST
- C12 pad 1: /ESP32-S3/3V3 -> VSS
- C13 pad 1: /ESP32-S3/3V3 -> 3V3
- C14 pad 1: /ESP32-S3/3V3 -> 3V3
- C5 pad 1: VSS -> 3V3
- C9 pad 1: VSS -> 3V3
- IC2 pad 16: VSS -> 3V3
- IC4 pad 8: VSS -> 3V3
- IC5 pad 10: /I5 -> /I6
- IC5 pad 11: /ESP32-S3/GPIO18 -> GND
- IC5 pad 12: /ESP32-S3/GPIO8 -> /EN3
- IC5 pad 13: /ESP32-S3/D- -> /I5
- IC5 pad 14: /ESP32-S3/D+ -> GND
- IC5 pad 15: /ESP32-S3/GPIO3 -> /SCL2
- IC5 pad 16: /ESP32-S3/GPIO46 -> /SDA2
- IC5 pad 17: /SCL2 -> /ESP32-C6/DR-
- IC5 pad 18: /SDA2 -> /ESP32-C6/DR+
- IC5 pad 19: /ESP32-S3/GPIO11 -> unconnected-(IC5-IO14-Pad19)
- IC5 pad 2: /ESP32-S3/3V3 -> GND
- IC5 pad 20: /ESP32-S3/GPIO12 -> /SCL
- IC5 pad 21: /SCL -> unconnected-(IC5-NC_3-Pad21)
- IC5 pad 23: /ESP32-S3/GPIO21 -> /ESP32-C6/BOOT
- IC5 pad 24: /ESP32-S3/GPIO47 -> /I4
- IC5 pad 25: /ESP32-S3/GPIO48 -> /EN2
- IC5 pad 26: /ESP32-S3/GPIO45 -> /I3
- IC5 pad 27: /ESP32-S3/BOOT -> /I2
- IC5 pad 28: /ESP32-S3/GPIO35 -> /EN1
- IC5 pad 29: /ESP32-S3/GPIO36 -> /I1
- IC5 pad 3: /ESP32-S3/RST -> 3V3
- IC5 pad 31: /I4 -> /ESP32-C6/GPIO16
- IC5 pad 32: /EN2 -> unconnected-(IC5-NC_4-Pad32)
- IC5 pad 33: /I3 -> unconnected-(IC5-NC_5-Pad33)
- IC5 pad 34: /I2 -> unconnected-(IC5-NC_6-Pad34)
- IC5 pad 35: /EN1 -> unconnected-(IC5-NC_7-Pad35)
- IC5 pad 36: /I1 -> GND
- IC5 pad 37: /ESP32-S3/GPIO43 -> GND
- IC5 pad 38: /ESP32-S3/GPIO2 -> GND
- IC5 pad 39: /ESP32-S3/GPIO1 -> GND
- IC5 pad 4: /ESP32-S3/GPIO4 -> unconnected-(IC5-NC_1-Pad4)
- IC5 pad 7: /I7 -> unconnected-(IC5-NC_2-Pad7)
- IC5 pad 8: /I6 -> /ESP32-C6/RST
- IC5 pad 9: /EN3 -> /I7
- J10 pad A6: /ESP32-S3/USB_D+ -> unconnected-(J10-D+-PadA6)
- J10 pad A7: /ESP32-S3/USB_D- -> unconnected-(J10-D--PadA7)
- J10 pad B6: /ESP32-S3/USB_D+ -> /ESP32-C6/USB_D+
- J10 pad B7: /ESP32-S3/USB_D- -> /ESP32-C6/USB_D-
- J4 pad 4: VSS -> 3V3
- J5 pad 4: VSS -> 3V3
- J6 pad 4: VSS -> 3V3
- J7 pad 4: VSS -> 3V3
- R10 pad 1: VSS -> 3V3
- R11 pad 1: VSS -> 3V3
- R12 pad 1: VSS -> 3V3
- R13 pad 1: VSS -> 3V3
- R14 pad 1: VSS -> 3V3
- R17 pad 1: VSS -> 3V3
- R19 pad 1: VSS -> 3V3
- R20 pad 1: /ESP32-S3/RST -> /ESP32-C6/RST
- R20 pad 2: /ESP32-S3/3V3 -> 3V3
- R22 pad 2: /ESP32-S3/3V3 -> 3V3
- R4 pad 1: VSS -> 3V3
- R5 pad 1: VSS -> 3V3
- R6 pad 1: VSS -> 3V3
- R7 pad 1: VSS -> 3V3
- R8 pad 1: VSS -> 3V3
- R9 pad 1: VSS -> 3V3
- SW1 pad 1: /ESP32-S3/RST -> /ESP32-C6/RST
- SW2 pad 1: /ESP32-S3/BOOT -> /ESP32-C6/BOOT
- U1 pad 1: /ESP32-S3/USB_D+ -> /ESP32-C6/USB_D-
- U1 pad 3: /ESP32-S3/USB_D- -> /ESP32-C6/USB_D+
- U1 pad 4: /ESP32-S3/D+ -> /ESP32-C6/D+
- U1 pad 6: /ESP32-S3/D- -> /ESP32-C6/D-
- U2 pad 2: /ESP32-S3/3V3 -> 3V3
Routing:
- net 3V3: track 0.00 -> 360.0 mm, vias 0 -> 13
- net VSS: track 188.5 -> 299.1 mm, vias 14 -> 6
- net /ESP32-S3/USB_D-: track 32.5 -> 0.00 mm
- net /ESP32-S3/USB_D+: track 32.4 -> 0.00 mm, vias 2 -> 0
- net /ESP32-C6/RST: track 0.00 -> 32.1 mm, vias 0 -> 2
- net /ESP32-S3/3V3: track 29.3 -> 0.00 mm, vias 2 -> 0
- net /ESP32-C6/DR+: track 0.00 -> 22.8 mm
- net /ESP32-C6/DR-: track 0.00 -> 22.1 mm
- net /ESP32-C6/USB_D+: track 0.00 -> 20.3 mm, vias 0 -> 2
- net /ESP32-C6/USB_D-: track 0.00 -> 19.7 mm, vias 0 -> 2
- net /ESP32-C6/BOOT: track 0.00 -> 17.8 mm
- net /ESP32-S3/BOOT: track 16.6 -> 0.00 mm
- net /ESP32-S3/RST: track 11.0 -> 0.00 mm
- net /ESP32-S3/D-: track 5.55 -> 0.00 mm
- net /ESP32-S3/D+: track 5.55 -> 0.00 mm
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- removed copper zone on B.Cu, net /ESP32-S3/3V3
- removed copper zone on B.Cu, net VSS
Other:
- board size 100 x 80 mm -> 100 x 74 mm
- board text added: "EN"
- board text added: "Motor Driver Board v2.1"
- board text added: "RST"
- board text removed: "Motor Driver Board v2.0B"
