File: PowerDistribution/PCB/POWER_OUT.kicad_sch (KiCad schematic)
At the start: 6 parts, among them IC5 SI4162DY-T1-GE3, J5 Conn_01x02

Commit message: Adds PDB v2.0
Parts:
- renumbered IC5 to IC8, J5 to J6, R11 to R19, R19 to R20, R12 to R21
Changed lines of the file:
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@@
 		(dnp no)
 		(fields_autoplaced yes)
-		(property "Reference" "#PWR042"
+		(property "Reference" "#PWR041"
 			(at 67.31 90.17 0)
 			(hide yes)
@@
 			(project "LabRover_PDB"
 				(path "/1fc67981-3095-4915-bfe8-a1a01c138c0d/3b63dde8-4127-4fac-864d-3d0d809a2669"
-					(reference "#PWR042")
+					(reference "#PWR041")
 					(unit 1)
 				)
 				(path "/1fc67981-3095-4915-bfe8-a1a01c138c0d/5fd8678a-e7cf-4b33-a902-f0f60064b221"
-					(reference "#PWR044")
+					(reference "#PWR045")
 					(unit 1)
 				)
 				(path "/1fc67981-3095-4915-bfe8-a1a01c138c0d/9557f421-8a47-48fc-b70a-dbac94f48fb3"
-					(reference "#PWR045")
+					(reference "#PWR047")
 					(unit 1)
 				)
@@
 		(in_pos_files yes)
 		(dnp no)
-		(property "Reference" "R12"
+		(property "Reference" "R21"
 			(at 106.6799 33.02 90)
 			(show_name no)
@@
 			(project "LabRover_PDB"
 				(path "/1fc67981-3095-4915-bfe8-a1a01c138c0d/3b63dde8-4127-4fac-864d-3d0d809a2669"
-					(reference "R12")
+					(reference "R21")
 					(unit 1)
 				)
 				(path "/1fc67981-3095-4915-bfe8-a1a01c138c0d/5fd8678a-e7cf-4b33-a902-f0f60064b221"
-					(reference "R16")
+					(reference "R27")
 					(unit 1)
 				)
 				(path "/1fc67981-3095-4915-bfe8-a1a01c138c0d/9557f421-8a47-48fc-b70a-dbac94f48fb3"
-					(reference "R18")
+					(reference "R30")
 					(unit 1)
 				)
 				(path "/1fc67981-3095-4915-bfe8-a1a01c138c0d/ae348767-f482-4f8b-b19d-e6b0836d928d"
-					(reference "R14")
+					(reference "R24")
 					(unit 1)
 				)
@@
 		(dnp no)
 		(fields_autoplaced yes)
-		(property "Reference" "#PWR035"
+		(property "Reference" "#PWR042"
 			(at 101.6 104.14 0)
 			(hide yes)
@@
 			(project "LabRover_PDB"
 				(path "/1fc67981-3095-4915-bfe8-a1a01c138c0d/3b63dde8-4127-4fac-864d-3d0d809a2669"
-					(reference "#PWR035")
+					(reference "#PWR042")
 					(unit 1)
 				)
 				(path "/1fc67981-3095-4915-bfe8-a1a01c138c0d/5fd8678a-e7cf-4b33-a902-f0f60064b221"
-					(reference "#PWR039")
+					(reference "#PWR046")
 					(unit 1)
 				)
 				(path "/1fc67981-3095-4915-bfe8-a1a01c138c0d/9557f421-8a47-48fc-b70a-dbac94f48fb3"
-					(reference "#PWR041")
+					(reference "#PWR048")
 					(unit 1)
 				)
 				(path "/1fc67981-3095-4915-bfe8-a1a01c138c0d/ae348767-f482-4f8b-b19d-e6b0836d928d"
-					(reference "#PWR037")
+					(reference "#PWR044")
 					(unit 1)
 				)
@@
 		(in_pos_files yes)
 		(dnp no)
-		(property "Reference" "R19"
+		(property "Reference" "R20"
 			(at 63.5001 77.47 90)
 			(show_name no)
@@
 			(project "LabRover_PDB"
 				(path "/1fc67981-3095-4915-bfe8-a1a01c138c0d/3b63dde8-4127-4fac-864d-3d0d809a2669"
-					(reference "R19")
+					(reference "R20")
 					(unit 1)
 				)
 				(path "/1fc67981-3095-4915-bfe8-a1a01c138c0d/5fd8678a-e7cf-4b33-a902-f0f60064b221"
-					(reference "R21")
+					(reference "R26")
 					(unit 1)
 				)
 				(path "/1fc67981-3095-4915-bfe8-a1a01c138c0d/9557f421-8a47-48fc-b70a-dbac94f48fb3"
-					(reference "R22")
+					(reference "R29")
 					(unit 1)
 				)
 				(path "/1fc67981-3095-4915-bfe8-a1a01c138c0d/ae348767-f482-4f8b-b19d-e6b0836d928d"
-					(reference "R20")
+					(reference "R23")
 					(unit 1)
 				)
@@
 		(in_pos_files yes)
 		(dnp no)
-		(property "Reference" "J5"
+		(property "Reference" "J6"
 			(at 73.66 30.4801 0)
 			(show_name no)
@@
 			(project "LabRover_PDB"
 				(path "/1fc67981-3095-4915-bfe8-a1a01c138c0d/3b63dde8-4127-4fac-864d-3d0d809a2669"
-					(reference "J5")
+					(reference "J6")
 					(unit 1)
 				)
 				(path "/1fc67981-3095-4915-bfe8-a1a01c138c0d/5fd8678a-e7cf-4b33-a902-f0f60064b221"
+					(reference "J8")
+					(unit 1)
+				)
+				(path "/1fc67981-3095-4915-bfe8-a1a01c138c0d/9557f421-8a47-48fc-b70a-dbac94f48fb3"
+					(reference "J9")
+					(unit 1)
+				)
+				(path "/1fc67981-3095-4915-bfe8-a1a01c138c0d/ae348767-f482-4f8b-b19d-e6b0836d928d"
 					(reference "J7")
-					(unit 1)
-				)
-				(path "/1fc67981-3095-4915-bfe8-a1a01c138c0d/9557f421-8a47-48fc-b70a-dbac94f48fb3"
-					(reference "J8")
-					(unit 1)
-				)
-				(path "/1fc67981-3095-4915-bfe8-a1a01c138c0d/ae348767-f482-4f8b-b19d-e6b0836d928d"
-					(reference "J6")
 					(unit 1)
 				)
@@
 		(in_pos_files yes)
 		(dnp no)
-		(property "Reference" "IC5"
+		(property "Reference" "IC8"
 			(at 81.28 58.42 90)
 			(show_name no)
@@
 			(project "LabRover_PDB"
 				(path "/1fc67981-3095-4915-bfe8-a1a01c138c0d/3b63dde8-4127-4fac-864d-3d0d809a2669"
-					(reference "IC5")
+					(reference "IC8")
 					(unit 1)
 				)
 				(path "/1fc67981-3095-4915-bfe8-a1a01c138c0d/5fd8678a-e7cf-4b33-a902-f0f60064b221"
-					(reference "IC7")
+					(reference "IC10")
 					(unit 1)
 				)
 				(path "/1fc67981-3095-4915-bfe8-a1a01c138c0d/9557f421-8a47-48fc-b70a-dbac94f48fb3"
-					(reference "IC8")
+					(reference "IC11")
 					(unit 1)
 				)
 				(path "/1fc67981-3095-4915-bfe8-a1a01c138c0d/ae348767-f482-4f8b-b19d-e6b0836d928d"
-					(reference "IC6")
+					(reference "IC9")
 					(unit 1)
 				)
@@
 		(in_pos_files yes)
 		(dnp no)
-		(property "Reference" "R11"
+		(property "Reference" "R19"
 			(at 49.53 76.1999 90)
 			(show_name no)
@@
 			(project "LabRover_PDB"
 				(path "/1fc67981-3095-4915-bfe8-a1a01c138c0d/3b63dde8-4127-4fac-864d-3d0d809a2669"
-					(reference "R11")
+					(reference "R19")
 					(unit 1)
 				)
 				(path "/1fc67981-3095-4915-bfe8-a1a01c138c0d/5fd8678a-e7cf-4b33-a902-f0f60064b221"
-					(reference "R15")
+					(reference "R25")
 					(unit 1)
 				)
 				(path "/1fc67981-3095-4915-bfe8-a1a01c138c0d/9557f421-8a47-48fc-b70a-dbac94f48fb3"
-					(reference "R17")
+					(reference "R28")
 					(unit 1)
 				)
 				(path "/1fc67981-3095-4915-bfe8-a1a01c138c0d/ae348767-f482-4f8b-b19d-e6b0836d928d"
-					(reference "R13")
-					(unit 1)
-				)
+					(reference "R22")
+					(unit 1)
+				)
