File: PowerDistribution/PCB/POWER_OUT.kicad_sch (KiCad schematic)
At the start: 6 parts, among them IC8 SI4162DY-T1-GE3, J6 Conn_01x02

Commit message: Gitignore fix
Parts:
- IC8: footprint SOIC127P600X175-8N -> Footprints:SI4162DY-T1-GE3
- J6: footprint Connector_AMASS:AMASS_XT30U-M_1x02_P5.0mm_Vertical -> Footprints:XT30
Changed lines of the file:
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@@
 			)
 		)
-		(property "Footprint" "Connector_AMASS:AMASS_XT30U-M_1x02_P5.0mm_Vertical"
+		(property "Footprint" "Footprints:XT30"
 			(at 76.2 30.48 0)
 			(hide yes)
@@
 			)
 		)
-		(property "Footprint" "SOIC127P600X175-8N"
+		(property "Footprint" "Footprints:SI4162DY-T1-GE3"
 			(at -2.21 50.8 0)
 			(hide yes)
