File: PowerDistribution/PCB/Power_Protection.kicad_sch (KiCad schematic)
At the start: 21 parts, among them IC1 TLV1117LV33DCYR, IC10 SI4162DY-T1-GE3, IC4 SN74LVC1G08DBVR, J1 Conn_01x02, J2 Conn_01x02, J3 Conn_01x02, J4 Conn_01x02, Q1 BSS84

Commit message: Adds PDB v2.0
Parts:
- renumbered D10 to D2, D9 to D3, D2 to D4, IC4 to IC1, IC10 to IC2, IC1 to IC3, J4 to J1, J1 to J2, J2 to J3, J3 to J4, R3 to R1, R28 to R3, R6 to R4, R23 to R5, R4 to R6
Changed lines of the file:
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@@
 		(dnp no)
 		(fields_autoplaced yes)
-		(property "Reference" "#PWR053"
+		(property "Reference" "#PWR03"
 			(at 35.56 55.88 0)
 			(hide yes)
@@
 			(project "LabRover_PDB"
 				(path "/1fc67981-3095-4915-bfe8-a1a01c138c0d/3886f5c7-0bd1-410a-a053-69be8d5593cb"
-					(reference "#PWR053")
+					(reference "#PWR03")
 					(unit 1)
 				)
@@
 		(in_pos_files yes)
 		(dnp no)
-		(property "Reference" "#PWR07"
+		(property "Reference" "#PWR09"
 			(at 93.98 109.22 0)
 			(hide yes)
@@
 			(project "LabRover_PDB"
 				(path "/1fc67981-3095-4915-bfe8-a1a01c138c0d/3886f5c7-0bd1-410a-a053-69be8d5593cb"
-					(reference "#PWR07")
+					(reference "#PWR09")
 					(unit 1)
 				)
@@
 		(dnp no)
 		(fields_autoplaced yes)
-		(property "Reference" "#PWR05"
+		(property "Reference" "#PWR06"
 			(at 55.88 133.35 0)
 			(hide yes)
@@
 			(project "LabRover_PDB"
 				(path "/1fc67981-3095-4915-bfe8-a1a01c138c0d/3886f5c7-0bd1-410a-a053-69be8d5593cb"
-					(reference "#PWR05")
+					(reference "#PWR06")
 					(unit 1)
 				)
@@
 		(dnp no)
 		(fields_autoplaced yes)
-		(property "Reference" "J2"
+		(property "Reference" "J3"
 			(at 34.29 111.7599 0)
 			(show_name no)
@@
 			(project "LabRover_PDB"
 				(path "/1fc67981-3095-4915-bfe8-a1a01c138c0d/3886f5c7-0bd1-410a-a053-69be8d5593cb"
-					(reference "J2")
+					(reference "J3")
 					(unit 1)
 				)
@@
 		(in_pos_files yes)
 		(dnp no)
-		(property "Reference" "D9"
+		(property "Reference" "D3"
 			(at 119.126 32.004 90)
 			(show_name no)
@@
 			(project "LabRover_PDB"
 				(path "/1fc67981-3095-4915-bfe8-a1a01c138c0d/3886f5c7-0bd1-410a-a053-69be8d5593cb"
-					(reference "D9")
+					(reference "D3")
 					(unit 1)
 				)
@@
 		(in_pos_files yes)
 		(dnp no)
-		(property "Reference" "J4"
+		(property "Reference" "J1"
 			(at 27.94 52.0699 0)
 			(hide yes)
@@
 			(project "LabRover_PDB"
 				(path "/1fc67981-3095-4915-bfe8-a1a01c138c0d/3886f5c7-0bd1-410a-a053-69be8d5593cb"
-					(reference "J4")
+					(reference "J1")
 					(unit 1)
 				)
@@
 		(in_pos_files yes)
 		(dnp no)
-		(property "Reference" "D2"
+		(property "Reference" "D4"
 			(at 207.518 144.018 90)
 			(show_name no)
@@
 			(project "LabRover_PDB"
 				(path "/1fc67981-3095-4915-bfe8-a1a01c138c0d/3886f5c7-0bd1-410a-a053-69be8d5593cb"
-					(reference "D2")
+					(reference "D4")
 					(unit 1)
 				)
@@
 		(dnp no)
 		(fields_autoplaced yes)
-		(property "Reference" "R3"
+		(property "Reference" "R1"
 			(at 58.42 114.3 0)
 			(show_name no)
@@
 			(project "LabRover_PDB"
 				(path "/1fc67981-3095-4915-bfe8-a1a01c138c0d/3886f5c7-0bd1-410a-a053-69be8d5593cb"
-					(reference "R3")
+					(reference "R1")
 					(unit 1)
 				)
@@
 		(dnp no)
 		(fields_autoplaced yes)
-		(property "Reference" "R6"
+		(property "Reference" "R4"
 			(at 106.68 116.84 0)
 			(show_name no)
@@
 			(project "LabRover_PDB"
 				(path "/1fc67981-3095-4915-bfe8-a1a01c138c0d/3886f5c7-0bd1-410a-a053-69be8d5593cb"
-					(reference "R6")
+					(reference "R4")
 					(unit 1)
 				)
@@
 		(dnp no)
 		(fields_autoplaced yes)
-		(property "Reference" "#PWR049"
+		(property "Reference" "#PWR08"
 			(at 86.36 71.12 0)
 			(hide yes)
@@
 			(project "LabRover_PDB"
 				(path "/1fc67981-3095-4915-bfe8-a1a01c138c0d/3886f5c7-0bd1-410a-a053-69be8d5593cb"
-					(reference "#PWR049")
+					(reference "#PWR08")
 					(unit 1)
 				)
@@
 		(dnp no)
 		(fields_autoplaced yes)
-		(property "Reference" "#PWR08"
+		(property "Reference" "#PWR012"
 			(at 119.38 154.94 0)
 			(hide yes)
@@
 			(project "LabRover_PDB"
 				(path "/1fc67981-3095-4915-bfe8-a1a01c138c0d/3886f5c7-0bd1-410a-a053-69be8d5593cb"
-					(reference "#PWR08")
+					(reference "#PWR012")
 					(unit 1)
 				)
@@
 		(dnp no)
 		(fields_autoplaced yes)
-		(property "Reference" "IC4"
+		(property "Reference" "IC1"
 			(at 54.61 44.45 0)
 			(show_name no)
@@
 			(project "LabRover_PDB"
 				(path "/1fc67981-3095-4915-bfe8-a1a01c138c0d/3886f5c7-0bd1-410a-a053-69be8d5593cb"
-					(reference "IC4")
+					(reference "IC1")
 					(unit 1)
 				)
@@
 		(dnp no)
 		(fields_autoplaced yes)
-		(property "Reference" "R4"
+		(property "Reference" "R6"
 			(at 201.93 135.89 0)
 			(show_name no)
@@
 			(project "LabRover_PDB"
 				(path "/1fc67981-3095-4915-bfe8-a1a01c138c0d/3886f5c7-0bd1-410a-a053-69be8d5593cb"
-					(reference "R4")
+					(reference "R6")
 					(unit 1)
 				)
@@
 		(dnp no)
 		(fields_autoplaced yes)
-		(property "Reference" "#PWR014"
+		(property "Reference" "#PWR016"
 			(at 199.39 154.94 0)
 			(hide yes)
@@
 			(project "LabRover_PDB"
 				(path "/1fc67981-3095-4915-bfe8-a1a01c138c0d/3886f5c7-0bd1-410a-a053-69be8d5593cb"
-					(reference "#PWR014")
+					(reference "#PWR016")
 					(unit 1)
 				)
@@
 		(in_pos_files yes)
 		(dnp no)
-		(property "Reference" "J3"
+		(property "Reference" "J4"
 			(at 34.29 25.4 0)
 			(show_name no)
@@
 			(project "LabRover_PDB"
 				(path "/1fc67981-3095-4915-bfe8-a1a01c138c0d/3886f5c7-0bd1-410a-a053-69be8d5593cb"
-					(reference "J3")
+					(reference "J4")
 					(unit 1)
 				)
@@
 		(dnp no)
 		(fields_autoplaced yes)
-		(property "Reference" "#PWR051"
+		(property "Reference" "#PWR04"
 			(at 41.91 68.58 0)
 			(hide yes)
@@
 			(project "LabRover_PDB"
 				(path "/1fc67981-3095-4915-bfe8-a1a01c138c0d/3886f5c7-0bd1-410a-a053-69be8d5593cb"
-					(reference "#PWR051")
+					(reference "#PWR04")
 					(unit 1)
 				)
@@
 		(dnp no)
 		(fields_autoplaced yes)
-		(property "Reference" "#PWR03"
+		(property "Reference" "#PWR011"
 			(at 116.84 68.58 0)
 			(hide yes)
@@
 			(project "LabRover_PDB"
 				(path "/1fc67981-3095-4915-bfe8-a1a01c138c0d/3886f5c7-0bd1-410a-a053-69be8d5593cb"
-					(reference "#PWR03")
+					(reference "#PWR011")
 					(unit 1)
 				)
@@
 		(in_pos_files yes)
 		(dnp no)
-		(property "Reference" "R28"
+		(property "Reference" "R3"
 			(at 82.5501 58.42 90)
 			(show_name no)
@@
 			(project "LabRover_PDB"
 				(path "/1fc67981-3095-4915-bfe8-a1a01c138c0d/3886f5c7-0bd1-410a-a053-69be8d5593cb"
-					(reference "R28")
+					(reference "R3")
 					(unit 1)
 				)
@@
 		(dnp no)
 		(fields_autoplaced yes)
-		(property "Reference" "IC1"
+		(property "Reference" "IC3"
 			(at 151.13 123.19 0)
 			(show_name no)
@@
 			(project "LabRover_PDB"
 				(path "/1fc67981-3095-4915-bfe8-a1a01c138c0d/3886f5c7-0bd1-410a-a053-69be8d5593cb"
-					(reference "IC1")
+					(reference "IC3")
 					(unit 1)
 				)
@@
 		(dnp no)
 		(fields_autoplaced yes)
-		(property "Reference" "#PWR052"
+		(property "Reference" "#PWR07"
 			(at 72.39 54.61 0)
 			(hide yes)
@@
 			(project "LabRover_PDB"
 				(path "/1fc67981-3095-4915-bfe8-a1a01c138c0d/3886f5c7-0bd1-410a-a053-69be8d5593cb"
-					(reference "#PWR052")
+					(reference "#PWR07")
 					(unit 1)
 				)
@@
 		(dnp no)
 		(fields_autoplaced yes)
-		(property "Reference" "#PWR09"
+		(property "Reference" "#PWR013"
 			(at 128.27 148.59 0)
 			(hide yes)
@@
 			(project "LabRover_PDB"
 				(path "/1fc67981-3095-4915-bfe8-a1a01c138c0d/3886f5c7-0bd1-410a-a053-69be8d5593cb"
-					(reference "#PWR09")
+					(reference "#PWR013")
 					(unit 1)
 				)
@@
 		(in_pos_files yes)
 		(dnp no)
-		(property "Reference" "IC10"
+		(property "Reference" "IC2"
 			(at 116.586 56.896 0)
 			(show_name no)
@@
 			(project "LabRover_PDB"
 				(path "/1fc67981-3095-4915-bfe8-a1a01c138c0d/3886f5c7-0bd1-410a-a053-69be8d5593cb"
-					(reference "IC10")
+					(reference "IC2")
 					(unit 1)
 				)
@@
 		(dnp no)
 		(fields_autoplaced yes)
-		(property "Reference" "#PWR011"
+		(property "Reference" "#PWR014"
 			(at 170.18 149.86 0)
 			(hide yes)
@@
 			(project "LabRover_PDB"
 				(path "/1fc67981-3095-4915-bfe8-a1a01c138c0d/3886f5c7-0bd1-410a-a053-69be8d5593cb"
-					(reference "#PWR011")
+					(reference "#PWR014")
 					(unit 1)
 				)
@@
 		(dnp no)
 		(fields_autoplaced yes)
-		(property "Reference" "#PWR06"
+		(property "Reference" "#PWR010"
 			(at 104.14 128.27 0)
 			(hide yes)
@@
 			(project "LabRover_PDB"
 				(path "/1fc67981-3095-4915-bfe8-a1a01c138c0d/3886f5c7-0bd1-410a-a053-69be8d5593cb"
-					(reference "#PWR06")
+					(reference "#PWR010")
 					(unit 1)
 				)
@@
 		(in_pos_files yes)
 		(dnp no)
-		(property "Reference" "R23"
+		(property "Reference" "R5"
 			(at 117.602 24.13 0)
 			(show_name no)
@@
 			(project "LabRover_PDB"
 				(path "/1fc67981-3095-4915-bfe8-a1a01c138c0d/3886f5c7-0bd1-410a-a053-69be8d5593cb"
-					(reference "R23")
+					(reference "R5")
 					(unit 1)
 				)
@@
 		(dnp no)
 		(fields_autoplaced yes)
-		(property "Reference" "#PWR050"
+		(property "Reference" "#PWR015"
 			(at 172.72 134.62 0)
 			(hide yes)
@@
 			(project "LabRover_PDB"
 				(path "/1fc67981-3095-4915-bfe8-a1a01c138c0d/3886f5c7-0bd1-410a-a053-69be8d5593cb"
-					(reference "#PWR050")
+					(reference "#PWR015")
 					(unit 1)
 				)
@@
 		(dnp no)
 		(fields_autoplaced yes)
-		(property "Reference" "#PWR04"
+		(property "Reference" "#PWR05"
 			(at 55.88 115.57 0)
 			(hide yes)
@@
 			(project "LabRover_PDB"
 				(path "/1fc67981-3095-4915-bfe8-a1a01c138c0d/3886f5c7-0bd1-410a-a053-69be8d5593cb"
-					(reference "#PWR04")
+					(reference "#PWR05")
 					(unit 1)
 				)
@@
 		(dnp no)
 		(fields_autoplaced yes)
-		(property "Reference" "D10"
+		(property "Reference" "D2"
 			(at 116.84 119.38 90)
 			(show_name no)
@@
 			(project "LabRover_PDB"
 				(path "/1fc67981-3095-4915-bfe8-a1a01c138c0d/3886f5c7-0bd1-410a-a053-69be8d5593cb"
-					(reference "D10")
+					(reference "D2")
 					(unit 1)
 				)
@@
 		(dnp no)
 		(fields_autoplaced yes)
-		(property "Reference" "J1"
+		(property "Reference" "J2"
 			(at 33.02 121.9199 0)
 			(show_name no)
@@
 			(project "LabRover_PDB"
 				(path "/1fc67981-3095-4915-bfe8-a1a01c138c0d/3886f5c7-0bd1-410a-a053-69be8d5593cb"
-					(reference "J1")
+					(reference "J2")
 					(unit 1)
 				)
