File: PowerDistribution/PCB/Sensors.kicad_sch (KiCad schematic)
At the start: 11 parts, among them IC2 LM75BDP,118, IC3 INA219AIDR, IC9 ADS1015BQDGSRQ1

Commit message: Adds PDB v2.0
Parts:
- renumbered C6 to C5, IC2 to IC4, IC3 to IC5, IC9 to IC6, R27 to R10, R10 to R11, R24 to R7, R26 to R8, R25 to R9
Changed lines of the file:
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@@
 		(dnp no)
 		(fields_autoplaced yes)
-		(property "Reference" "IC9"
+		(property "Reference" "IC6"
 			(at 194.31 80.01 0)
 			(show_name no)
@@
 			(project "LabRover_PDB"
 				(path "/1fc67981-3095-4915-bfe8-a1a01c138c0d/0940b463-1e23-448c-ab36-d79df28b12e9"
-					(reference "IC9")
+					(reference "IC6")
 					(unit 1)
 				)
@@
 		(dnp no)
 		(fields_autoplaced yes)
-		(property "Reference" "#PWR046"
+		(property "Reference" "#PWR030"
 			(at 229.87 96.52 0)
 			(hide yes)
@@
 			(project "LabRover_PDB"
 				(path "/1fc67981-3095-4915-bfe8-a1a01c138c0d/0940b463-1e23-448c-ab36-d79df28b12e9"
-					(reference "#PWR046")
+					(reference "#PWR030")
 					(unit 1)
 				)
@@
 		(dnp no)
 		(fields_autoplaced yes)
-		(property "Reference" "R27"
+		(property "Reference" "R10"
 			(at 147.32 88.9 0)
 			(show_name no)
@@
 			(project "LabRover_PDB"
 				(path "/1fc67981-3095-4915-bfe8-a1a01c138c0d/0940b463-1e23-448c-ab36-d79df28b12e9"
-					(reference "R27")
+					(reference "R10")
 					(unit 1)
 				)
@@
 		(dnp no)
 		(fields_autoplaced yes)
-		(property "Reference" "#PWR021"
+		(property "Reference" "#PWR022"
 			(at 165.1 46.99 0)
 			(hide yes)
@@
 			(project "LabRover_PDB"
 				(path "/1fc67981-3095-4915-bfe8-a1a01c138c0d/0940b463-1e23-448c-ab36-d79df28b12e9"
-					(reference "#PWR021")
+					(reference "#PWR022")
 					(unit 1)
 				)
@@
 		(dnp no)
 		(fields_autoplaced yes)
-		(property "Reference" "R10"
+		(property "Reference" "R11"
 			(at 210.82 41.9099 0)
 			(show_name no)
@@
 			(project "LabRover_PDB"
 				(path "/1fc67981-3095-4915-bfe8-a1a01c138c0d/0940b463-1e23-448c-ab36-d79df28b12e9"
-					(reference "R10")
+					(reference "R11")
 					(unit 1)
 				)
@@
 		(dnp no)
 		(fields_autoplaced yes)
-		(property "Reference" "IC3"
+		(property "Reference" "IC5"
 			(at 184.15 36.83 0)
 			(show_name no)
@@
 			(project "LabRover_PDB"
 				(path "/1fc67981-3095-4915-bfe8-a1a01c138c0d/0940b463-1e23-448c-ab36-d79df28b12e9"
-					(reference "IC3")
+					(reference "IC5")
 					(unit 1)
 				)
@@
 		(dnp no)
 		(fields_autoplaced yes)
-		(property "Reference" "#PWR019"
+		(property "Reference" "#PWR020"
 			(at 130.81 52.07 0)
 			(hide yes)
@@
 			(project "LabRover_PDB"
 				(path "/1fc67981-3095-4915-bfe8-a1a01c138c0d/0940b463-1e23-448c-ab36-d79df28b12e9"
-					(reference "#PWR019")
+					(reference "#PWR020")
 					(unit 1)
 				)
@@
 		(in_pos_files yes)
 		(dnp no)
-		(property "Reference" "#PWR038"
+		(property "Reference" "#PWR023"
 			(at 171.45 110.49 0)
 			(hide yes)
@@
 			(project "LabRover_PDB"
 				(path "/1fc67981-3095-4915-bfe8-a1a01c138c0d/0940b463-1e23-448c-ab36-d79df28b12e9"
-					(reference "#PWR038")
+					(reference "#PWR023")
 					(unit 1)
 				)
@@
 		(dnp no)
 		(fields_autoplaced yes)
-		(property "Reference" "#PWR036"
+		(property "Reference" "#PWR018"
 			(at 116.84 100.33 0)
 			(hide yes)
@@
 			(project "LabRover_PDB"
 				(path "/1fc67981-3095-4915-bfe8-a1a01c138c0d/0940b463-1e23-448c-ab36-d79df28b12e9"
-					(reference "#PWR036")
+					(reference "#PWR018")
 					(unit 1)
 				)
@@
 		(dnp no)
 		(fields_autoplaced yes)
-		(property "Reference" "#PWR018"
+		(property "Reference" "#PWR019"
 			(at 130.81 41.91 0)
 			(hide yes)
@@
 			(project "LabRover_PDB"
 				(path "/1fc67981-3095-4915-bfe8-a1a01c138c0d/0940b463-1e23-448c-ab36-d79df28b12e9"
-					(reference "#PWR018")
+					(reference "#PWR019")
 					(unit 1)
 				)
@@
 		(in_pos_files yes)
 		(dnp no)
-		(property "Reference" "#PWR047"
+		(property "Reference" "#PWR031"
 			(at 229.87 106.68 0)
 			(hide yes)
@@
 			(project "LabRover_PDB"
 				(path "/1fc67981-3095-4915-bfe8-a1a01c138c0d/0940b463-1e23-448c-ab36-d79df28b12e9"
-					(reference "#PWR047")
+					(reference "#PWR031")
 					(unit 1)
 				)
@@
 		(dnp no)
 		(fields_autoplaced yes)
-		(property "Reference" "R26"
+		(property "Reference" "R8"
 			(at 119.38 88.9 0)
 			(show_name no)
@@
 			(project "LabRover_PDB"
 				(path "/1fc67981-3095-4915-bfe8-a1a01c138c0d/0940b463-1e23-448c-ab36-d79df28b12e9"
-					(reference "R26")
+					(reference "R8")
 					(unit 1)
 				)
@@
 		(dnp no)
 		(fields_autoplaced yes)
-		(property "Reference" "#PWR048"
+		(property "Reference" "#PWR021"
 			(at 144.78 100.33 0)
 			(hide yes)
@@
 			(project "LabRover_PDB"
 				(path "/1fc67981-3095-4915-bfe8-a1a01c138c0d/0940b463-1e23-448c-ab36-d79df28b12e9"
-					(reference "#PWR048")
+					(reference "#PWR021")
 					(unit 1)
 				)
@@
 		(in_pos_files yes)
 		(dnp no)
-		(property "Reference" "R24"
+		(property "Reference" "R7"
 			(at 111.76 82.296 90)
 			(show_name no)
@@
 			(project "LabRover_PDB"
 				(path "/1fc67981-3095-4915-bfe8-a1a01c138c0d/0940b463-1e23-448c-ab36-d79df28b12e9"
-					(reference "R24")
+					(reference "R7")
 					(unit 1)
 				)
@@
 		(in_pos_files yes)
 		(dnp no)
-		(property "Reference" "R25"
+		(property "Reference" "R9"
 			(at 139.7 82.296 90)
 			(show_name no)
@@
 			(project "LabRover_PDB"
 				(path "/1fc67981-3095-4915-bfe8-a1a01c138c0d/0940b463-1e23-448c-ab36-d79df28b12e9"
-					(reference "R25")
+					(reference "R9")
 					(unit 1)
 				)
@@
 		(dnp no)
 		(fields_autoplaced yes)
-		(property "Reference" "C6"
+		(property "Reference" "C5"
 			(at 233.68 95.2499 0)
 			(show_name no)
@@
 			(project "LabRover_PDB"
 				(path "/1fc67981-3095-4915-bfe8-a1a01c138c0d/0940b463-1e23-448c-ab36-d79df28b12e9"
-					(reference "C6")
+					(reference "C5")
 					(unit 1)
 				)
@@
 		(dnp no)
 		(fields_autoplaced yes)
-		(property "Reference" "#PWR040"
+		(property "Reference" "#PWR024"
 			(at 176.53 91.44 0)
 			(hide yes)
@@
 			(project "LabRover_PDB"
 				(path "/1fc67981-3095-4915-bfe8-a1a01c138c0d/0940b463-1e23-448c-ab36-d79df28b12e9"
-					(reference "#PWR040")
+					(reference "#PWR024")
 					(unit 1)
 				)
@@
 		(dnp no)
 		(fields_autoplaced yes)
-		(property "Reference" "IC2"
+		(property "Reference" "IC4"
 			(at 106.68 30.48 0)
 			(show_name no)
@@
 			(project "LabRover_PDB"
 				(path "/1fc67981-3095-4915-bfe8-a1a01c138c0d/0940b463-1e23-448c-ab36-d79df28b12e9"
-					(reference "IC2")
-					(unit 1)
-				)
+					(reference "IC4")
+					(unit 1)
+				)
