File: PowerDistribution/PCB/LabRover_PDB.kicad_pcb (KiCad board)
At the start: 4 copper layers, 79 x 67 mm, 75 parts, among them IC1 SN74LVC1G08DBVR, IC10 SI4162DY-T1-GE3, IC11 SI4162DY-T1-GE3, IC2 SI4162DY-T1-GE3, IC3 TLV1117LV33DCYR, IC4 LM75BDP,118, IC5 INA219AIDR, IC6 ADS1015BQDGSRQ1, IC7 ESP32-C3-MINI-1U-N4X, IC8 SI4162DY-T1-GE3, IC9 SI4162DY-T1-GE3, J1 Conn_01x02, J2 Conn_01x02, J3 Conn_01x02, J4 Conn_01x02, J5 USB_C_Receptacle_USB2.0_16P, J6 Conn_01x02, J7 Conn_01x02, J8 Conn_01x02, J9 Conn_01x02, Q1 BSS84, SW1 SW_Push, SW2 SW_Push, U1 USBLC6-2SC6

Commit message: Firmware for v2.0, and hardware fixes change for v2.1
Parts:
- added R31: 10k, Resistor_SMD:R_0402_1005Metric, F.Cu at (148.0, 99.0)
- added R32: 10k, Resistor_SMD:R_0402_1005Metric, F.Cu at (141.5, 97.0)
- added R33: 10k, Resistor_SMD:R_0402_1005Metric, F.Cu at (172.5, 94.0)
- added R34: 10k, Resistor_SMD:R_0402_1005Metric, F.Cu at (173.5, 94.0)
Routing:
- net GND: track 88.4 -> 92.1 mm, vias 34 -> 241
- net /ESP32_C3/GPIO1: track 6.47 -> 10.1 mm
- net +3.3V: track 141.5 -> 143.6 mm, vias 7 -> 8
- net /ESP32_C3/GPIO20: track 61.8 -> 63.6 mm, vias 4 -> 5
- net Net-(IC1-B): track 20.4 -> 22.2 mm, vias 1 -> 2
- net /ESP32_C3/GPIO21: track 64.4 -> 65.5 mm, vias 4 -> 5
Other:
- board text added: "Odyssey PDB V2.1"
- board text removed: "Odyssey PDB V2.0"

Commit message: Gitignore fix
Parts:
- C1, C2: footprint Footprints:CAPPM3528X210N -> Footprints:TAJB226K020RNJ
- IC1: footprint Footprints:SOT95P280X145-5N -> Footprints:SN74LVC1G08DBVR
- IC10, IC11, IC2, IC8, IC9: footprint Footprints:SOIC127P600X175-8N -> Footprints:SI4162DY-T1-GE3
- IC3: footprint Footprints:SOT230P700X180-4N -> Package_TO_SOT_SMD:SOT-223-3_TabPin2
- IC4: footprint Footprints:SOP65P490X110-8N -> Footprints:LM75BDP,118
- IC5: footprint Footprints:SOIC127P600X175-8N -> Footprints:INA219AIDR
- IC6: footprint Footprints:SOP50P490X110-10N -> Footprints:ADS1015BQDGSRQ1
- J4: footprint Connector_AMASS:AMASS_XT90PW-M_1x02_P10.90mm_Horizontal -> Footprints:AMASS_XT90PW-M
- J5: footprint Connector_USB:USB_C_Receptacle_G-Switch_GT-USB-7010ASV -> Footprints:USB_C_Receptacle_G-Switch_GT-USB-7010ASV
- J6, J7, J8, J9: footprint Connector_AMASS:AMASS_XT30U-M_1x02_P5.0mm_Vertical -> Footprints:XT30
- moved J4 10.9 mm to (124.0, 106.6), turned to -90 degrees
