File: PowerDistribution/PCB/uC.kicad_sch (KiCad schematic)
At the start: 15 parts, among them IC7 ESP32-C3-MINI-1U-N4X, J5 USB_C_Receptacle_USB2.0_16P, SW1 SW_Push, SW2 SW_Push, U1 USBLC6-2SC6

Commit message: Gitignore fix
Parts:
- IC7: footprint ESP32C3MINI1UN4X -> Footprints:ESP32C3MINI1UN4X
- J5: footprint Connector_USB:USB_C_Receptacle_G-Switch_GT-USB-7010ASV -> Footprints:USB_C_Receptacle_G-Switch_GT-USB-7010ASV
Changed lines of the file:
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@@
 			)
 		)
-		(property "Footprint" "ESP32C3MINI1UN4X"
+		(property "Footprint" "Footprints:ESP32C3MINI1UN4X"
 			(at 254 129.21 0)
 			(hide yes)
@@
 			)
 		)
-		(property "Footprint" "Connector_USB:USB_C_Receptacle_G-Switch_GT-USB-7010ASV"
+		(property "Footprint" "Footprints:USB_C_Receptacle_G-Switch_GT-USB-7010ASV"
 			(at 68.58 57.15 0)
 			(hide yes)
